File: battery_powered_temp_logger.sch (KiCad schematic (older format))
At the start: 6 parts, among them U6 DS18B20, U7 ESP-201

Commit message: restore symbol table
Parts:
- U7: symbol ESP8266:ESP-201 -> iothome-rescue:ESP-201-ESP8266
Changed lines of the file:
@@
 EESchema Schematic File Version 4
 LIBS:iothome-cache
-EELAYER 26 0
+EELAYER 29 0
 EELAYER END
 $Descr A4 11693 8268
@@
 $EndDescr
 $Comp
-L ESP8266:ESP-201 U7
+L iothome-rescue:ESP-201-ESP8266 U7
 U 1 1 5C44522F
 P 5200 3750
+AR Path="/5C44522F" Ref="U7"  Part="1"
+AR Path="/5C4451C9/5C44522F" Ref="U7"  Part="1"
 F 0 "U7" H 5200 2978 50  0000 C CNN
 F 1 "ESP-201" H 5200 2887 50  0000 C CNN
