File: iothome.sch (KiCad schematic (older format))
At the start: 14 parts, among them J1 USB_B, J2 USB_A, U1 BA033ST, U2 ESP-01, U3 AP1117-33, U4 ESP-01, U5 DS18B20

Commit message: restore symbol table
Parts:
- U1: symbol rohm_ba033st:BA033ST -> iothome-rescue:BA033ST-rohm_ba033st
- U2, U4: symbol ESP8266_modules:ESP-01 -> iothome-rescue:ESP-01-ESP8266_modules
Changed lines of the file:
@@
 EESchema Schematic File Version 4
 LIBS:iothome-cache
-EELAYER 26 0
+EELAYER 29 0
 EELAYER END
 $Descr A4 11693 8268
@@
 	2400 2550 3200 2550
 $Comp
-L rohm_ba033st:BA033ST U1
+L iothome-rescue:BA033ST-rohm_ba033st U1
 U 1 1 5C3BBD10
 P 3200 1850
@@
 	3200 2550 4000 2550
 $Comp
-L ESP8266_modules:ESP-01 U2
+L iothome-rescue:ESP-01-ESP8266_modules U2
 U 1 1 5C3BCC0E
 P 4800 1550
@@
 Connection ~ 2600 5000
 $Comp
-L ESP8266_modules:ESP-01 U4
+L iothome-rescue:ESP-01-ESP8266_modules U4
 U 1 1 5C3C1924
 P 4200 4000
